Commit message: configure the urdf files to correct package name

File: omnibot_ws/src/omnibot_description/urdf/base_link.urdf.xacro (robot description, xacro)
@@ -1,13 +1,13 @@
 <?xml version="1.0"?>
 <robot xmlns:xacro="http://ros.org/wiki/xacro">
-  <xacro:include filename="$(find ros2_omni_robot_sim)/urdf/3w_v2/omni_wheel.urdf.xacro"/>
-  <xacro:include filename="$(find ros2_omni_robot_sim)/urdf/3w_v2/camera.urdf.xacro"/>
-  <xacro:include filename="$(find ros2_omni_robot_sim)/urdf/3w_v2/lidar.urdf.xacro"/>
-  <xacro:include filename="$(find ros2_omni_robot_sim)/urdf/3w_v2/imu.urdf.xacro"/>
+  <xacro:include filename="$(find omnibot_description)/urdf/omni_wheel.urdf.xacro"/>
+  <xacro:include filename="$(find omnibot_description)/urdf/camera.urdf.xacro"/>
+  <xacro:include filename="$(find omnibot_description)/urdf/lidar.urdf.xacro"/>
+  <xacro:include filename="$(find omnibot_description)/urdf/imu.urdf.xacro"/>
   <xacro:macro name="base_link" params="parent xyz rpy">
     <link name="base_link">
       <visual>
         <geometry>
-          <mesh filename="package://ros2_omni_robot_sim/meshes/3w_v2/base_link.dae" />
+          <mesh filename="package://omnibot_description/meshes/3w_v2/base_link.dae" />
         </geometry>
         <!-- <material name="base_color">
@@ -17,5 +17,5 @@
       <collision>
         <geometry>
-          <mesh filename="package://ros2_omni_robot_sim/meshes/3w_v2/base_link.stl" />
+          <mesh filename="package://omnibot_description/meshes/3w_v2/base_link.stl" />
         </geometry>
       </collision>

File: omnibot_ws/src/omnibot_description/urdf/camera.urdf.xacro (robot description, xacro)
@@ -5,5 +5,5 @@
       <visual>
         <geometry>
-          <mesh filename="package://ros2_omni_robot_sim/meshes/3w_v2/camera.stl" />
+          <mesh filename="package://omnibot_description/meshes/3w_v2/camera.stl" />
         </geometry>
         <material name="black">
@@ -13,5 +13,5 @@
       <collision>
         <geometry>
-          <mesh filename="package://ros2_omni_robot_sim/meshes/3w_v2/camera.stl" />
+          <mesh filename="package://omnibot_description/meshes/3w_v2/camera.stl" />
         </geometry>
       </collision>

File: omnibot_ws/src/omnibot_description/urdf/gazebo_plugins.urdf.xacro (robot description, xacro)
@@ -8,5 +8,5 @@
     <plugin name="ignition::gazebo::systems::Imu" filename="libignition-gazebo-imu-system.so" />
     <plugin filename="ign_ros2_control-system" name="ign_ros2_control::IgnitionROS2ControlPlugin">
-      <parameters>$(find ros2_omni_robot_sim)/config/controller_configs/controller_config_3w_v2.yaml</parameters>
+      <parameters>$(find omnibot_controllers)/config/controller_configs/controller_config_3w_v2.yaml</parameters>
     </plugin>
   </gazebo>

File: omnibot_ws/src/omnibot_description/urdf/main.urdf.xacro (robot description, xacro)
@@ -1,7 +1,7 @@
 <?xml version="1.0"?>
 <robot name="simple_robot" xmlns:xacro="http://ros.org/wiki/xacro">
-  <xacro:include filename="$(find ros2_omni_robot_sim)/urdf/3w_v2/base_link.urdf.xacro" />
-  <xacro:include filename="$(find ros2_omni_robot_sim)/urdf/3w_v2/gazebo_plugins.urdf.xacro" />
-  <xacro:include filename="$(find ros2_omni_robot_sim)/urdf/3w_v2/ros2_control.urdf.xacro" />
+  <xacro:include filename="$(find omnibot_description)/urdf/base_link.urdf.xacro" />
+  <xacro:include filename="$(find omnibot_description)/urdf/gazebo_plugins.urdf.xacro" />
+  <xacro:include filename="$(find omnibot_description)/urdf/ros2_control.urdf.xacro" />
   <link name="base_footprint" />
   <!-- Base Link -->

File: omnibot_ws/src/omnibot_description/urdf/omni_wheel.urdf.xacro (robot description, xacro)
@@ -1,10 +1,10 @@
 <?xml version="1.0"?>
 <robot xmlns:xacro="http://ros.org/wiki/xacro">
-  <xacro:include filename="$(find ros2_omni_robot_sim)/urdf/3w_v2/roller.urdf.xacro"/>
+  <xacro:include filename="$(find omnibot_description)/urdf/roller.urdf.xacro"/>
   <xacro:macro name="omni_wheel" params="suffix parent xyz rpy">
     <link name="omni_wheel_link_${suffix}">
       <visual>
         <geometry>
-          <mesh filename="package://ros2_omni_robot_sim/meshes/3w_v2/omni_frame.stl" />
+          <mesh filename="package://omnibot_description/meshes/3w_v2/omni_frame.stl" />
         </geometry>
         <material name="white">
@@ -14,5 +14,5 @@
       <collision>
         <geometry>
-          <mesh filename="package://ros2_omni_robot_sim/meshes/3w_v2/omni_frame.stl" />
+          <mesh filename="package://omnibot_description/meshes/3w_v2/omni_frame.stl" />
         </geometry>
       </collision>

File: omnibot_ws/src/omnibot_description/urdf/roller.urdf.xacro (robot description, xacro)
@@ -5,5 +5,5 @@
       <visual>
         <geometry>
-          <mesh filename="package://ros2_omni_robot_sim/meshes/3w_v2/roller.stl" />
+          <mesh filename="package://omnibot_description/meshes/3w_v2/roller.stl" />
         </geometry>
         <material name="black">
@@ -13,5 +13,5 @@
       <collision>
         <geometry>
-          <mesh filename="package://ros2_omni_robot_sim/meshes/3w_v2/roller.stl" />
+          <mesh filename="package://omnibot_description/meshes/3w_v2/roller.stl" />
         </geometry>
       </collision>

Commit message: add launch for controller

File: omnibot_ws/src/omnibot_description/urdf/base_link.urdf.xacro (robot description, xacro)
@@ -16,6 +16,7 @@
       </visual>
       <collision>
+        <origin xyz="0 0 0.05" rpy="0 0 0"/>
         <geometry>
-          <mesh filename="package://omnibot_description/meshes/3w_v2/base_link.stl" />
+          <cylinder radius="0.125" length="0.09"/>
         </geometry>
       </collision>
